Commit message: enable spawning multiple robots from xacro

File: xacro/barista_robot_model.xacro (robot description, xacro)
@@ -5,5 +5,15 @@
   <xacro:include filename="$(find barista_robot_description)/xacro/cup_holder_tray.xacro" />
   <xacro:arg name="include_laser" default="true"/>
-    <material name="gray">
+  <xacro:arg name="robot_name" default=""/>
+  <xacro:arg name="color" default="blue"/>
+  <xacro:property name="robot_name" value="$(arg robot_name)"/>
+  <xacro:property name="color" value="$(arg color)"/>
+  <xacro:if value="${robot_name == ''}">
+    <xacro:property name="prefix" value=""/>
+  </xacro:if>
+  <xacro:unless value="${robot_name == ''}">
+    <xacro:property name="prefix" value="${robot_name}_"/>
+  </xacro:unless>
+  <material name="gray">
       <color rgba="0.5 0.5 0.5 1"/>
   </material>
@@ -11,65 +21,78 @@
       <color rgba="0.0 0.0 1.0 1"/>
   </material>
+  <material name="red">
+      <color rgba="1.0 0.0 0.0 1"/>
+  </material>
   <material name="black">
       <color rgba="0.0 0.0 0.0 1"/>
   </material>
-  <link name="base_link">
-  </link>
-  <joint name="base_link_to_chassis" type="fixed">
+  <link name="${prefix}base_link">
+  </link>
+  <joint name="${prefix}base_link_to_chassis" type="fixed">
     <origin rpy="0 0 0" xyz="0 0 0" />
-    <parent link="base_link"/>
-    <child link="chassis"/>
-  </joint>
-  <gazebo reference="chassis">
-    <material>Gazebo/Blue</material>
-  </gazebo>
-  <link name="chassis">
-    <visual>
-      <origin rpy="0 0 0" xyz="0 0 0"/>
-      <geometry>
-        <cylinder length="0.155" radius="0.178"/>
-      </geometry>
-      <material name="blue"/>
-    </visual>
-    <collision>
-      <origin rpy="0 0 0" xyz="0 0 0"/>
-      <geometry>
-        <cylinder length="0.155" radius="0.178"/>
-      </geometry>
-    </collision>
-    <inertial>
-      <origin rpy="0 0 0" xyz="0 0 0"/>
-      <mass value="5"/>
-      <inertia ixx="0.04961541666666667" ixy="0.0" ixz="0.0" iyy="0.04961541666666667" iyz="0.0" izz="0.07920999999999999"/>
-    </inertial>
-  </link>
-  <joint name="chassis_to_left_wheel" type="continuous">
+    <parent link="${prefix}base_link"/>
+    <child link="${prefix}chassis"/>
+  </joint>
+  <xacro:macro name="chassis" params="color name">
+    <xacro:if value="${color == 'blue'}">
+      <gazebo reference="${name}">
+        <material>Gazebo/Blue</material>
+      </gazebo>
+    </xacro:if>
+    <xacro:if value="${color == 'red'}">
+      <gazebo reference="${name}">
+        <material>Gazebo/Red</material>
+      </gazebo>
+    </xacro:if>
+    <link name="${name}">
+      <visual>
+        <origin rpy="0 0 0" xyz="0 0 0"/>
+        <geometry>
+          <cylinder length="0.155" radius="0.178"/>
+        </geometry>
+        <material name="${color}"/>
+      </visual>
+      <collision>
+        <origin rpy="0 0 0" xyz="0 0 0"/>
+        <geometry>
+          <cylinder length="0.155" radius="0.178"/>
+        </geometry>
+      </collision>
+      <inertial>
+        <origin rpy="0 0 0" xyz="0 0 0"/>
+        <mass value="5"/>
+        <inertia ixx="0.04961541666666667" ixy="0.0" ixz="0.0" iyy="0.04961541666666667" iyz="0.0" izz="0.07920999999999999"/>
+      </inertial>
+    </link>
+  </xacro:macro>
+  <xacro:chassis name="${prefix}chassis" color="${color}"/>
+  <joint name="${prefix}chassis_to_left_wheel" type="continuous">
     <origin rpy="0 -1.57 0" xyz="-0.150 0.0 -0.0775"/>
-    <parent link="chassis"/>
-    <child link="left_wheel"/>
+    <parent link="${prefix}chassis"/>
+    <child link="${prefix}left_wheel"/>
     <axis rpy="0 0 0" xyz="0 0 1"/>
     <limit effort="10000" velocity="1000"/>
     <joint_properties damping="1.0" friction="1.0"/>
   </joint>
-  <xacro:wheel wheel_name="left_wheel" />
-  <joint name="chassis_to_right_wheel" type="continuous">
+  <xacro:wheel wheel_name="${prefix}left_wheel" />
+  <joint name="${prefix}chassis_to_right_wheel" type="continuous">
     <origin rpy="0 -1.57 0" xyz="0.150 0.0 -0.0775"/>
-    <parent link="chassis"/>
-    <child link="right_wheel"/>
+    <parent link="${prefix}chassis"/>
+    <child link="${prefix}right_wheel"/>
     <axis rpy="0 0 0" xyz="0 0 1"/>
     <limit effort="10000" velocity="1000"/>
     <joint_properties damping="1.0" friction="1.0"/>
   </joint>
-  <xacro:wheel wheel_name="right_wheel" />
+  <xacro:wheel wheel_name="${prefix}right_wheel" />
   <!-- Caster Wheel Front -->
-  <joint name="front_yaw_joint" type="continuous">
+  <joint name="${prefix}front_yaw_joint" type="continuous">
     <origin rpy="0 0 0" xyz="0.0 0.130 -0.0775" />
-    <parent link="chassis" />
-    <child link="front_yaw_link" />
+    <parent link="${prefix}chassis" />
+    <child link="${prefix}front_yaw_link" />
     <axis xyz="0 0 1" />
     <limit effort="1000.0" velocity="100.0" />
     <dynamics damping="0.0" friction="0.1"/>
   </joint>
-  <link name="front_yaw_link">
+  <link name="${prefix}front_yaw_link">
       <visual>
         <origin rpy="0 1.5707 1.5707" xyz="0 0 0"/>
@@ -91,13 +114,13 @@
       </inertial>
   </link>
-  <joint name="front_roll_joint" type="continuous">
+  <joint name="${prefix}front_roll_joint" type="continuous">
     <origin rpy="0 0 0" xyz="0 0 0" />
-    <parent link="front_yaw_link" />
-    <child link="front_roll_link" />
+    <parent link="${prefix}front_yaw_link" />
+    <child link="${prefix}front_roll_link" />
     <axis xyz="1 0 0" />
     <limit effort="1000.0" velocity="100.0" />
     <dynamics damping="0.0" friction="0.1"/>
   </joint>
-  <link name="front_roll_link">
+  <link name="${prefix}front_roll_link">
       <visual>
         <origin rpy="0 1.5707 1.5707" xyz="0 0 0"/>
@@ -119,13 +142,13 @@
       </inertial>
   </link>
-  <joint name="front_pitch_joint" type="continuous">
+  <joint name="${prefix}front_pitch_joint" type="continuous">
     <origin rpy="0 0 0" xyz="0 0 0" />
-    <parent link="front_roll_link" />
-    <child link="front_pitch_link" />
+    <parent link="${prefix}front_roll_link" />
+    <child link="${prefix}front_pitch_link" />
     <axis xyz="0 1 0" />
     <limit effort="1000.0" velocity="100.0" />
     <dynamics damping="0.0" friction="0.1"/>
   </joint>
-  <gazebo reference="front_pitch_link">
+  <gazebo reference="{prefix}front_pitch_link">
     <kp>1000000000000000000000000000.0</kp>
     <kd>1000000000000000000000000000.0</kd>
@@ -134,5 +157,5 @@
     <material>Gazebo/Black</material>
   </gazebo>
-  <link name="front_pitch_link">
+  <link name="${prefix}front_pitch_link">
     <visual>
       <origin rpy="0 1.5707 1.5707" xyz="0 0 0"/>
@@ -155,13 +178,13 @@
   </link>
   <!-- Caster Wheel Back -->
-  <joint name="back_yaw_joint" type="continuous">
+  <joint name="${prefix}back_yaw_joint" type="continuous">
     <origin rpy="0 0 0" xyz="0.0 -0.130 -0.0775" />
-    <parent link="chassis" />
-    <child link="back_yaw_link" />
+    <parent link="${prefix}chassis" />
+    <child link="${prefix}back_yaw_link" />
     <axis xyz="0 0 1" />
     <limit effort="1000.0" velocity="100.0" />
     <dynamics damping="0.0" friction="0.1"/>
   </joint>
-  <link name="back_yaw_link">
+  <link name="${prefix}back_yaw_link">
       <visual>
         <origin rpy="0 1.5707 1.5707" xyz="0 0 0"/>
@@ -183,13 +206,13 @@
       </inertial>
   </link>
-  <joint name="back_roll_joint" type="continuous">
+  <joint name="${prefix}back_roll_joint" type="continuous">
     <origin rpy="0 0 0" xyz="0 0 0" />
-    <parent link="back_yaw_link" />
-    <child link="back_roll_link" />
+    <parent link="${prefix}back_yaw_link" />
+    <child link="${prefix}back_roll_link" />
     <axis xyz="1 0 0" />
     <limit effort="1000.0" velocity="100.0" />
     <dynamics damping="0.0" friction="0.1"/>
   </joint>
-  <link name="back_roll_link">
+  <link name="${prefix}back_roll_link">
       <visual>
         <origin rpy="0 1.5707 1.5707" xyz="0 0 0"/>
@@ -211,13 +234,13 @@
       </inertial>
   </link>
-  <joint name="back_pitch_joint" type="continuous">
+  <joint name="${prefix}back_pitch_joint" type="continuous">
     <origin rpy="0 0 0" xyz="0 0 0" />
-    <parent link="back_roll_link" />
-    <child link="back_pitch_link" />
+    <parent link="${prefix}back_roll_link" />
+    <child link="${prefix}back_pitch_link" />
     <axis xyz="0 1 0" />
     <limit effort="1000.0" velocity="100.0" />
     <dynamics damping="0.0" friction="0.1"/>
   </joint>
-  <gazebo reference="back_pitch_link">
+  <gazebo reference="{prefix}back_pitch_link">
     <kp>1000000000000000000000000000.0</kp>
     <kd>1000000000000000000000000000.0</kd>
@@ -226,5 +249,5 @@
     <material>Gazebo/Black</material>
   </gazebo>
-  <link name="back_pitch_link">
+  <link name="${prefix}back_pitch_link">
     <visual>
       <origin rpy="0 1.5707 1.5707" xyz="0 0 0"/>
@@ -246,41 +269,41 @@
     </inertial>
   </link>
-  <joint name="chassis_to_cup_holder_tray" type="fixed">
+  <joint name="${prefix}chassis_to_cup_holder_tray" type="fixed">
     <origin rpy="0 0 0" xyz="0 0 0.3425" />
-    <parent link="base_link"/>
-    <child link="cup_holder_tray"/>
-  </joint>
-  <xacro:cup_holder_tray/>
-  <joint name="chassis_to_standoff_rod_back_left" type="fixed">
+    <parent link="${prefix}base_link"/>
+    <child link="${prefix}cup_holder_tray"/>
+  </joint>
+  <xacro:cup_holder_tray cup_holder_tray_name="${prefix}cup_holder_tray" color="${color}"/>
+  <joint name="${prefix}chassis_to_standoff_rod_back_left" type="fixed">
     <origin rpy="0 0 0" xyz="-0.140 -0.030 0.1875" />
-    <parent link="chassis"/>
-    <child link="standoff_rod_back_left"/>
-  </joint>
-  <xacro:standoff standoff_name="standoff_rod_back_left"/>
-  <joint name="chassis_to_standoff_rod_back_right" type="fixed">
+    <parent link="${prefix}chassis"/>
+    <child link="${prefix}standoff_rod_back_left"/>
+  </joint>
+  <xacro:standoff standoff_name="${prefix}standoff_rod_back_left"/>
+  <joint name="${prefix}chassis_to_standoff_rod_back_right" type="fixed">
     <origin rpy="0 0 0" xyz="0.140 -0.030 0.1875" />
-    <parent link="chassis"/>
-    <child link="standoff_rod_back_right"/>
-  </joint>
-  <xacro:standoff standoff_name="standoff_rod_back_right"/>
-  <joint name="chassis_to_standoff_rod_front_left" type="fixed">
+    <parent link="${prefix}chassis"/>
+    <child link="${prefix}standoff_rod_back_right"/>
+  </joint>
+  <xacro:standoff standoff_name="${prefix}standoff_rod_back_right"/>
+  <joint name="${prefix}chassis_to_standoff_rod_front_left" type="fixed">
     <origin rpy="0 0 0" xyz="-0.140 0.030 0.1875"/>
-    <parent link="chassis"/>
-    <child link="standoff_rod_front_left"/>
-  </joint>
-  <xacro:standoff standoff_name="standoff_rod_front_left"/>
-  <joint name="chassis_to_standoff_rod_front_right" type="fixed">
+    <parent link="${prefix}chassis"/>
+    <child link="${prefix}standoff_rod_front_left"/>
+  </joint>
+  <xacro:standoff standoff_name="${prefix}standoff_rod_front_left"/>
+  <joint name="${prefix}chassis_to_standoff_rod_front_right" type="fixed">
     <origin rpy="0 0 0" xyz="0.140 0.030 0.1875"/>
-    <parent link="chassis"/>
-    <child link="standoff_rod_front_right"/>
-  </joint>
-  <xacro:standoff standoff_name="standoff_rod_front_right"/>
+    <parent link="${prefix}chassis"/>
+    <child link="${prefix}standoff_rod_front_right"/>
+  </joint>
+  <xacro:standoff standoff_name="${prefix}standoff_rod_front_right"/>
   <!--Laser-->
-  <joint name="chassis_to_laser_scan_link" type="fixed">
+  <joint name="${prefix}chassis_to_laser_scan_link" type="fixed">
     <origin rpy="0 0 0" xyz="0.0 0.0 0.0775"/>
-    <parent link="chassis"/>
-    <child link="laser_scan_link"/>
-  </joint>
-  <link name="laser_scan_link">
+    <parent link="${prefix}chassis"/>
+    <child link="${prefix}laser_scan_link"/>
+  </joint>
+  <link name="${prefix}laser_scan_link">
     <visual>
       <origin rpy="0 0 1.57" xyz="0 0 0"/>
@@ -304,14 +327,14 @@
     </inertial>
   </link>
-  <joint name="laser_scan_link_to_laser_scan_frame" type="fixed">
+  <joint name="${prefix}laser_scan_link_to_laser_scan_frame" type="fixed">
     <origin rpy="0 0 1.57" xyz="0 0 0.08"/>
-    <parent link="laser_scan_link"/>
-    <child link="laser_scan_frame"/>
-  </joint>
-  <link name="laser_scan_frame">
+    <parent link="${prefix}laser_scan_link"/>
+    <child link="${prefix}laser_scan_frame"/>
+  </joint>
+  <link name="${prefix}laser_scan_frame">
   </link>
   <xacro:macro name="laser" params="include_laser">
     <xacro:if value="${include_laser}">
-      <gazebo reference="laser_scan_frame">
+      <gazebo reference="${prefix}laser_scan_frame">
         <sensor name="sensor_ray" type="ray">
           <pose>0 0 0 0 0 0</pose>
@@ -335,4 +358,5 @@
           <plugin name="laser" filename="libgazebo_ros_ray_sensor.so">
             <ros>
+              <namespace>/${robot_name}</namespace>
               <remapping>~/out:=scan</remapping>
             </ros>
@@ -348,15 +372,16 @@
     <plugin name="barista_robot_joint_state" filename="libgazebo_ros_joint_state_publisher.so">
       <ros>
+          <namespace>/${robot_name}</namespace>
           <remapping>~/out:=joint_states</remapping>
       </ros>
       <update_rate>30</update_rate>
-      <joint_name>chassis_to_left_wheel</joint_name>
-      <joint_name>chassis_to_right_wheel</joint_name>
-      <joint_name>front_yaw_joint</joint_name>
-      <joint_name>front_roll_joint</joint_name>
-      <joint_name>front_pitch_joint</joint_name>
-      <joint_name>back_yaw_joint</joint_name>
-      <joint_name>back_roll_joint</joint_name>
-      <joint_name>back_pitch_joint</joint_name>
+      <joint_name>${prefix}chassis_to_left_wheel</joint_name>
+      <joint_name>${prefix}chassis_to_right_wheel</joint_name>
+      <joint_name>${prefix}front_yaw_joint</joint_name>
+      <joint_name>${prefix}front_roll_joint</joint_name>
+      <joint_name>${prefix}front_pitch_joint</joint_name>
+      <joint_name>${prefix}back_yaw_joint</joint_name>
+      <joint_name>${prefix}back_roll_joint</joint_name>
+      <joint_name>${prefix}back_pitch_joint</joint_name>
     </plugin>
   </gazebo>
@@ -364,7 +389,11 @@
   <gazebo>
     <plugin filename="libgazebo_ros_diff_drive.so" name="differential_drive_controller">
+      <ros>
+        <namespace>/${robot_name}</namespace>
+        <remapping>/cmd_vel:=cmd_vel</remapping>
+      </ros>
       <!-- wheels -->
-      <left_joint>chassis_to_left_wheel</left_joint>
-      <right_joint>chassis_to_right_wheel</right_joint>
+      <left_joint>${prefix}chassis_to_left_wheel</left_joint>
+      <right_joint>${prefix}chassis_to_right_wheel</right_joint>
       <!-- kinematics -->
       <wheel_separation>0.300</wheel_separation>
@@ -376,6 +405,6 @@
       <publish_odom>true</publish_odom>
       <publish_odom_tf>true</publish_odom_tf>
-      <odometry_frame>odom</odometry_frame>
-      <robot_base_frame>base_link</robot_base_frame>
+      <odometry_frame>${prefix}odom</odometry_frame>
+      <robot_base_frame>${prefix}base_link</robot_base_frame>
     </plugin>
   </gazebo>

File: xacro/cup_holder_tray.xacro (robot description, xacro)
@@ -1,8 +1,15 @@
 <?xml version="1.0"?>
 <robot xmlns:xacro="http://www.ros.org/wiki/xacro">
-<xacro:macro name="cup_holder_tray" params="cup_holder_tray_name:=cup_holder_tray">
-  <gazebo reference="${cup_holder_tray_name}">
-    <material>Gazebo/Blue</material>
-  </gazebo>
+<xacro:macro name="cup_holder_tray" params="cup_holder_tray_name:=cup_holder_tray color:=blue">
+  <xacro:if value="${color == 'blue'}">
+    <gazebo reference="${cup_holder_tray_name}">
+      <material>Gazebo/Blue</material>
+    </gazebo>
+  </xacro:if>
+  <xacro:if value="${color == 'red'}">
+    <gazebo reference="${cup_holder_tray_name}">
+      <material>Gazebo/Red</material>
+    </gazebo>
+  </xacro:if>
   <link name="${cup_holder_tray_name}">
     <visual>
@@ -11,5 +18,5 @@
         <cylinder length="0.090" radius="0.160"/>
       </geometry>
-      <material name="blue"/>
+      <material name="${color}"/>
     </visual>
     <collision>
