Commit message: implement visual, collision and physical barista robot model

File: urdf/barista_robot_model.urdf (robot description, URDF)
Before this commit: robot barista_robot, 1 links, 0 joints
Links:
- added link back_pitch_link, mass 0.001; collision sphere radius=0.0352; visual sphere radius=0.0352
- added link back_roll_link, mass 0.001; collision cylinder length=0.001 radius=0.0045000000000000005; visual cylinder length=0.001 radius=0.0045000000000000005
- added link back_yaw_link, mass 0.001; collision cylinder length=0.001 radius=0.0045000000000000005; visual cylinder length=0.001 radius=0.0045000000000000005
- added link base_link
- added link cup_holder_tray, mass 1.0; collision cylinder length=0.090 radius=0.160; visual cylinder length=0.090 radius=0.160
- added link front_pitch_link, mass 0.001; collision sphere radius=0.0352; visual sphere radius=0.0352
- added link front_roll_link, mass 0.001; collision cylinder length=0.001 radius=0.0045000000000000005; visual cylinder length=0.001 radius=0.0045000000000000005
- added link front_yaw_link, mass 0.001; collision cylinder length=0.001 radius=0.0045000000000000005; visual cylinder length=0.001 radius=0.0045000000000000005
- added link left_wheel, mass 0.05; collision cylinder length=0.0206 radius=0.0352; visual cylinder length=0.0206 radius=0.0352
- added link right_wheel, mass 0.05; collision cylinder length=0.0206 radius=0.0352; visual cylinder length=0.0206 radius=0.0352
- added link standoff_rod_back_left, mass 0.5; collision cylinder length=0.220 radius=0.010; visual cylinder length=0.220 radius=0.010
- added link standoff_rod_back_right, mass 0.5; collision cylinder length=0.220 radius=0.010; visual cylinder length=0.220 radius=0.010
- added link standoff_rod_front_left, mass 0.5; collision cylinder length=0.220 radius=0.010; visual cylinder length=0.220 radius=0.010
- added link standoff_rod_front_right, mass 0.5; collision cylinder length=0.220 radius=0.010; visual cylinder length=0.220 radius=0.010
- link chassis: mass 0.5 -> 5; geometry collision cylinder length=0.155 radius=0.178; visual cylinder length=0.155 radius=0.178
Joints:
- added joint back_pitch_joint: type continuous, parent back_roll_link, child back_pitch_link, origin xyz=0 0 0 rpy=0 0 0, axis 0 1 0, limit effort=1000.0 velocity=100.0
- added joint back_roll_joint: type continuous, parent back_yaw_link, child back_roll_link, origin xyz=0 0 0 rpy=0 0 0, axis 1 0 0, limit effort=1000.0 velocity=100.0
- added joint back_yaw_joint: type continuous, parent chassis, child back_yaw_link, origin xyz=0.0 -0.130 -0.0775 rpy=0 0 0, axis 0 0 1, limit effort=1000.0 velocity=100.0
- added joint base_link_to_chassis: type fixed, parent base_link, child chassis, origin xyz=0 0 0 rpy=0 0 0
- added joint chassis_to_cup_holder_tray: type fixed, parent base_link, child cup_holder_tray, origin xyz=0 0 0.3425 rpy=0 0 0
- added joint chassis_to_left_wheel: type continuous, parent chassis, child left_wheel, origin xyz=-0.150 0.0 -0.0775 rpy=0 -1.57 0, axis 0 0 1, limit effort=10000 velocity=1000
- added joint chassis_to_right_wheel: type continuous, parent chassis, child right_wheel, origin xyz=0.150 0.0 -0.0775 rpy=0 -1.57 0, axis 0 0 1, limit effort=10000 velocity=1000
- added joint chassis_to_standoff_rod_back_left: type fixed, parent chassis, child standoff_rod_back_left, origin xyz=-0.140 -0.030 0.1875 rpy=0 0 0
- added joint chassis_to_standoff_rod_back_right: type fixed, parent chassis, child standoff_rod_back_right, origin xyz=0.140 -0.030 0.1875 rpy=0 0 0
- added joint chassis_to_standoff_rod_front_left: type fixed, parent chassis, child standoff_rod_front_left, origin xyz=-0.140 0.030 0.1875 rpy=0 0 0
- added joint chassis_to_standoff_rod_front_right: type fixed, parent chassis, child standoff_rod_front_right, origin xyz=0.140 0.030 0.1875 rpy=0 0 0
- added joint front_pitch_joint: type continuous, parent front_roll_link, child front_pitch_link, origin xyz=0 0 0 rpy=0 0 0, axis 0 1 0, limit effort=1000.0 velocity=100.0
- added joint front_roll_joint: type continuous, parent front_yaw_link, child front_roll_link, origin xyz=0 0 0 rpy=0 0 0, axis 1 0 0, limit effort=1000.0 velocity=100.0
- added joint front_yaw_joint: type continuous, parent chassis, child front_yaw_link, origin xyz=0.0 0.130 -0.0775 rpy=0 0 0, axis 0 0 1, limit effort=1000.0 velocity=100.0

Commit message: add laser scanner

File: urdf/barista_robot_model.urdf (robot description, URDF)
Before this commit: robot barista_robot, 15 links, 14 joints
Links:
- added link laser_scan_frame
- added link laser_scan_link, mass 0.8; collision box size=0.08 0.08 0.095; visual mesh filename=package://barista_robot_description/meshes/hokuyo_uam05lp.d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 scale=1.0 1.0 1.0
Joints:
- added joint chassis_to_laser_scan_link: type fixed, parent chassis, child laser_scan_link, origin xyz=0.0 0.0 0.0775 rpy=0 0 0
- added joint laser_scan_link_to_laser_scan_frame: type fixed, parent laser_scan_link, child laser_scan_frame, origin xyz=0 0 0.08 rpy=0 0 1.57

Commit message: make x axis of base_link point forward

File: urdf/barista_robot_model.urdf (robot description, URDF)
Before this commit: robot barista_robot, 17 links, 16 joints
Joints:
- joint back_yaw_joint: origin xyz=0.0 -0.130 -0.0775 rpy=0 0 0 -> xyz=-0.130 0.0 -0.0775 rpy=0 0 0
- joint chassis_to_left_wheel: origin xyz=-0.150 0.0 -0.0775 rpy=0 -1.57 0 -> xyz=0.0 0.150 -0.0775 rpy=-1.57 0 0
- joint chassis_to_right_wheel: origin xyz=0.150 0.0 -0.0775 rpy=0 -1.57 0 -> xyz=0.0 -0.150 -0.0775 rpy=-1.57 0 0
- joint chassis_to_standoff_rod_back_left: origin xyz=-0.140 -0.030 0.1875 rpy=0 0 0 -> xyz=-0.030 0.140 0.1875 rpy=0 0 0
- joint chassis_to_standoff_rod_back_right: origin xyz=0.140 -0.030 0.1875 rpy=0 0 0 -> xyz=-0.030 -0.140 0.1875 rpy=0 0 0
- joint chassis_to_standoff_rod_front_left: origin xyz=-0.140 0.030 0.1875 rpy=0 0 0 -> xyz=0.030 0.140 0.1875 rpy=0 0 0
- joint chassis_to_standoff_rod_front_right: origin xyz=0.140 0.030 0.1875 rpy=0 0 0 -> xyz=0.030 -0.140 0.1875 rpy=0 0 0
- joint front_yaw_joint: origin xyz=0.0 0.130 -0.0775 rpy=0 0 0 -> xyz=0.130 0.0 -0.0775 rpy=0 0 0
- joint laser_scan_link_to_laser_scan_frame: origin xyz=0 0 0.08 rpy=0 0 1.57 -> xyz=0 0 0.08 rpy=0 0 0

File: xacro/barista_robot_model.xacro (robot description, xacro)
@@ -68,5 +68,5 @@
   <xacro:chassis name="${prefix}chassis" color="${color}"/>
   <joint name="${prefix}chassis_to_left_wheel" type="continuous">
-    <origin rpy="0 -1.57 0" xyz="-0.150 0.0 -0.0775"/>
+    <origin rpy="-1.57 0 0" xyz="0.0 0.150 -0.0775"/>
     <parent link="${prefix}chassis"/>
     <child link="${prefix}left_wheel"/>
@@ -77,5 +77,5 @@
   <xacro:wheel wheel_name="${prefix}left_wheel" />
   <joint name="${prefix}chassis_to_right_wheel" type="continuous">
-    <origin rpy="0 -1.57 0" xyz="0.150 0.0 -0.0775"/>
+    <origin rpy="-1.57 0 0" xyz="0.0 -0.150 -0.0775"/>
     <parent link="${prefix}chassis"/>
     <child link="${prefix}right_wheel"/>
@@ -87,5 +87,5 @@
   <!-- Caster Wheel Front -->
   <joint name="${prefix}front_yaw_joint" type="continuous">
-    <origin rpy="0 0 0" xyz="0.0 0.130 -0.0775" />
+    <origin rpy="0 0 0" xyz="0.130 0.0 -0.0775" />
     <parent link="${prefix}chassis" />
     <child link="${prefix}front_yaw_link" />
@@ -179,5 +179,5 @@
   <!-- Caster Wheel Back -->
   <joint name="${prefix}back_yaw_joint" type="continuous">
-    <origin rpy="0 0 0" xyz="0.0 -0.130 -0.0775" />
+    <origin rpy="0 0 0" xyz="-0.130 0.0 -0.0775" />
     <parent link="${prefix}chassis" />
     <child link="${prefix}back_yaw_link" />
@@ -276,5 +276,5 @@
   <xacro:cup_holder_tray cup_holder_tray_name="${prefix}cup_holder_tray" color="${color}"/>
   <joint name="${prefix}chassis_to_standoff_rod_back_left" type="fixed">
-    <origin rpy="0 0 0" xyz="-0.140 -0.030 0.1875" />
+    <origin rpy="0 0 0" xyz="-0.030 0.140 0.1875" />
     <parent link="${prefix}chassis"/>
     <child link="${prefix}standoff_rod_back_left"/>
@@ -282,5 +282,5 @@
   <xacro:standoff standoff_name="${prefix}standoff_rod_back_left"/>
   <joint name="${prefix}chassis_to_standoff_rod_back_right" type="fixed">
-    <origin rpy="0 0 0" xyz="0.140 -0.030 0.1875" />
+    <origin rpy="0 0 0" xyz="-0.030 -0.140 0.1875" />
     <parent link="${prefix}chassis"/>
     <child link="${prefix}standoff_rod_back_right"/>
@@ -288,5 +288,5 @@
   <xacro:standoff standoff_name="${prefix}standoff_rod_back_right"/>
   <joint name="${prefix}chassis_to_standoff_rod_front_left" type="fixed">
-    <origin rpy="0 0 0" xyz="-0.140 0.030 0.1875"/>
+    <origin rpy="0 0 0" xyz="0.030 0.140 0.1875"/>
     <parent link="${prefix}chassis"/>
     <child link="${prefix}standoff_rod_front_left"/>
@@ -294,5 +294,5 @@
   <xacro:standoff standoff_name="${prefix}standoff_rod_front_left"/>
   <joint name="${prefix}chassis_to_standoff_rod_front_right" type="fixed">
-    <origin rpy="0 0 0" xyz="0.140 0.030 0.1875"/>
+    <origin rpy="0 0 0" xyz="0.030 -0.140 0.1875"/>
     <parent link="${prefix}chassis"/>
     <child link="${prefix}standoff_rod_front_right"/>
@@ -307,5 +307,5 @@
   <link name="${prefix}laser_scan_link">
     <visual>
-      <origin rpy="0 0 1.57" xyz="0 0 0"/>
+      <origin rpy="0 0 0" xyz="0 0 0"/>
       <geometry>
         <mesh filename="package://barista_robot_description/meshes/hokuyo_uam05lp.dae" scale="1.0 1.0 1.0"/>
@@ -313,5 +313,5 @@
     </visual>
     <collision>
-      <origin rpy="0 0 1.57" xyz="0 0 0"/>
+      <origin rpy="0 0 0" xyz="0 0 0"/>
       <geometry>
         <!--from datasheet-->
@@ -328,5 +328,5 @@
   </link>
   <joint name="${prefix}laser_scan_link_to_laser_scan_frame" type="fixed">
-    <origin rpy="0 0 1.57" xyz="0 0 0.08"/>
+    <origin rpy="0 0 0" xyz="0 0 0.08"/>
     <parent link="${prefix}laser_scan_link"/>
     <child link="${prefix}laser_scan_frame"/>

Commit message: make x axis of base_link point forward

File: urdf/barista_robot_model.urdf (robot description, URDF)
Before this commit: robot barista_robot, 17 links, 16 joints
Joints:
- joint back_yaw_joint: origin xyz=0.0 -0.130 -0.0775 rpy=0 0 0 -> xyz=-0.130 0.0 -0.0775 rpy=0 0 0
- joint chassis_to_laser_scan_link: origin xyz=0.0 0.0 0.0775 rpy=0 0 0 -> xyz=0.0 0.0 0.0775 rpy=0 0 3.14
- joint chassis_to_left_wheel: origin xyz=-0.150 0.0 -0.0775 rpy=0 -1.57 0 -> xyz=0.0 0.150 -0.0775 rpy=1.57 0 0
- joint chassis_to_right_wheel: origin xyz=0.150 0.0 -0.0775 rpy=0 -1.57 0 -> xyz=0.0 -0.150 -0.0775 rpy=1.57 0 0
- joint chassis_to_standoff_rod_back_left: origin xyz=-0.140 -0.030 0.1875 rpy=0 0 0 -> xyz=-0.030 0.140 0.1875 rpy=0 0 0
- joint chassis_to_standoff_rod_back_right: origin xyz=0.140 -0.030 0.1875 rpy=0 0 0 -> xyz=-0.030 -0.140 0.1875 rpy=0 0 0
- joint chassis_to_standoff_rod_front_left: origin xyz=-0.140 0.030 0.1875 rpy=0 0 0 -> xyz=0.030 0.140 0.1875 rpy=0 0 0
- joint chassis_to_standoff_rod_front_right: origin xyz=0.140 0.030 0.1875 rpy=0 0 0 -> xyz=0.030 -0.140 0.1875 rpy=0 0 0
- joint front_yaw_joint: origin xyz=0.0 0.130 -0.0775 rpy=0 0 0 -> xyz=0.130 0.0 -0.0775 rpy=0 0 0
- joint laser_scan_link_to_laser_scan_frame: origin xyz=0 0 0.08 rpy=0 0 1.57 -> xyz=0 0 0.08 rpy=0 0 0

File: xacro/barista_robot_model.xacro (robot description, xacro)
@@ -68,5 +68,5 @@
   <xacro:chassis name="${prefix}chassis" color="${color}"/>
   <joint name="${prefix}chassis_to_left_wheel" type="continuous">
-    <origin rpy="0 -1.57 0" xyz="-0.150 0.0 -0.0775"/>
+    <origin rpy="1.57 0 0" xyz="0.0 0.150 -0.0775"/>
     <parent link="${prefix}chassis"/>
     <child link="${prefix}left_wheel"/>
@@ -77,5 +77,5 @@
   <xacro:wheel wheel_name="${prefix}left_wheel" />
   <joint name="${prefix}chassis_to_right_wheel" type="continuous">
-    <origin rpy="0 -1.57 0" xyz="0.150 0.0 -0.0775"/>
+    <origin rpy="1.57 0 0" xyz="0.0 -0.150 -0.0775"/>
     <parent link="${prefix}chassis"/>
     <child link="${prefix}right_wheel"/>
@@ -87,5 +87,5 @@
   <!-- Caster Wheel Front -->
   <joint name="${prefix}front_yaw_joint" type="continuous">
-    <origin rpy="0 0 0" xyz="0.0 0.130 -0.0775" />
+    <origin rpy="0 0 0" xyz="0.130 0.0 -0.0775" />
     <parent link="${prefix}chassis" />
     <child link="${prefix}front_yaw_link" />
@@ -179,5 +179,5 @@
   <!-- Caster Wheel Back -->
   <joint name="${prefix}back_yaw_joint" type="continuous">
-    <origin rpy="0 0 0" xyz="0.0 -0.130 -0.0775" />
+    <origin rpy="0 0 0" xyz="-0.130 0.0 -0.0775" />
     <parent link="${prefix}chassis" />
     <child link="${prefix}back_yaw_link" />
@@ -276,5 +276,5 @@
   <xacro:cup_holder_tray cup_holder_tray_name="${prefix}cup_holder_tray" color="${color}"/>
   <joint name="${prefix}chassis_to_standoff_rod_back_left" type="fixed">
-    <origin rpy="0 0 0" xyz="-0.140 -0.030 0.1875" />
+    <origin rpy="0 0 0" xyz="-0.030 0.140 0.1875" />
     <parent link="${prefix}chassis"/>
     <child link="${prefix}standoff_rod_back_left"/>
@@ -282,5 +282,5 @@
   <xacro:standoff standoff_name="${prefix}standoff_rod_back_left"/>
   <joint name="${prefix}chassis_to_standoff_rod_back_right" type="fixed">
-    <origin rpy="0 0 0" xyz="0.140 -0.030 0.1875" />
+    <origin rpy="0 0 0" xyz="-0.030 -0.140 0.1875" />
     <parent link="${prefix}chassis"/>
     <child link="${prefix}standoff_rod_back_right"/>
@@ -288,5 +288,5 @@
   <xacro:standoff standoff_name="${prefix}standoff_rod_back_right"/>
   <joint name="${prefix}chassis_to_standoff_rod_front_left" type="fixed">
-    <origin rpy="0 0 0" xyz="-0.140 0.030 0.1875"/>
+    <origin rpy="0 0 0" xyz="0.030 0.140 0.1875"/>
     <parent link="${prefix}chassis"/>
     <child link="${prefix}standoff_rod_front_left"/>
@@ -294,5 +294,5 @@
   <xacro:standoff standoff_name="${prefix}standoff_rod_front_left"/>
   <joint name="${prefix}chassis_to_standoff_rod_front_right" type="fixed">
-    <origin rpy="0 0 0" xyz="0.140 0.030 0.1875"/>
+    <origin rpy="0 0 0" xyz="0.030 -0.140 0.1875"/>
     <parent link="${prefix}chassis"/>
     <child link="${prefix}standoff_rod_front_right"/>
@@ -301,5 +301,5 @@
   <!--Laser-->
   <joint name="${prefix}chassis_to_laser_scan_link" type="fixed">
-    <origin rpy="0 0 0" xyz="0.0 0.0 0.0775"/>
+    <origin rpy="0 0 3.14" xyz="0.0 0.0 0.0775"/>
     <parent link="${prefix}chassis"/>
     <child link="${prefix}laser_scan_link"/>
@@ -307,5 +307,5 @@
   <link name="${prefix}laser_scan_link">
     <visual>
-      <origin rpy="0 0 1.57" xyz="0 0 0"/>
+      <origin rpy="0 0 0" xyz="0 0 0"/>
       <geometry>
         <mesh filename="package://barista_robot_description/meshes/hokuyo_uam05lp.dae" scale="1.0 1.0 1.0"/>
@@ -313,5 +313,5 @@
     </visual>
     <collision>
-      <origin rpy="0 0 1.57" xyz="0 0 0"/>
+      <origin rpy="0 0 0" xyz="0 0 0"/>
       <geometry>
         <!--from datasheet-->
@@ -328,5 +328,5 @@
   </link>
   <joint name="${prefix}laser_scan_link_to_laser_scan_frame" type="fixed">
-    <origin rpy="0 0 1.57" xyz="0 0 0.08"/>
+    <origin rpy="0 0 0" xyz="0 0 0.08"/>
     <parent link="${prefix}laser_scan_link"/>
     <child link="${prefix}laser_scan_frame"/>
